Commit message: redefine lidar pos

File: panther_sensor_kit_description/urdf/sensor_kit.xacro (robot description, xacro)
@@ -30,24 +30,4 @@
       />
     </xacro:VLP-16>
-    <!-- <xacro:VLP-16 parent="sensor_kit_base_link" name="velodyne_left" topic="/points_raw" hz="10" samples="220" gpu="$(arg gpu)">
-      <origin
-        xyz="${calibration['sensor_kit_base_link']['velodyne_left_base_link']['x']}
-             ${calibration['sensor_kit_base_link']['velodyne_left_base_link']['y']}
-             ${calibration['sensor_kit_base_link']['velodyne_left_base_link']['z']}"
-        rpy="${calibration['sensor_kit_base_link']['velodyne_left_base_link']['roll']}
-             ${calibration['sensor_kit_base_link']['velodyne_left_base_link']['pitch']}
-             ${calibration['sensor_kit_base_link']['velodyne_left_base_link']['yaw']}"
-      />
-    </xacro:VLP-16>
-    <xacro:VLP-16 parent="sensor_kit_base_link" name="velodyne_right" topic="/points_raw" hz="10" samples="220" gpu="$(arg gpu)">
-      <origin
-        xyz="${calibration['sensor_kit_base_link']['velodyne_right_base_link']['x']}
-             ${calibration['sensor_kit_base_link']['velodyne_right_base_link']['y']}
-             ${calibration['sensor_kit_base_link']['velodyne_right_base_link']['z']}"
-        rpy="${calibration['sensor_kit_base_link']['velodyne_right_base_link']['roll']}
-             ${calibration['sensor_kit_base_link']['velodyne_right_base_link']['pitch']}
-             ${calibration['sensor_kit_base_link']['velodyne_right_base_link']['yaw']}"
-      />
-    </xacro:VLP-16> -->
     <!-- camera -->
     <!-- <xacro:monocular_camera_macro
@@ -67,5 +47,5 @@
     /> -->
     <!-- gnss -->
-    <xacro:imu_macro
+    <!-- <xacro:imu_macro
       name="gnss"
       parent="sensor_kit_base_link"
@@ -78,7 +58,7 @@
       yaw="${calibration['sensor_kit_base_link']['gnss_link']['yaw']}"
       fps="100"
-    />
+    /> -->
     <!-- imu -->
-    <xacro:imu_macro
+    <!-- <xacro:imu_macro
       name="tamagawa/imu"
       parent="sensor_kit_base_link"
@@ -91,5 +71,5 @@
       yaw="${calibration['sensor_kit_base_link']['tamagawa/imu_link']['yaw']}"
       fps="100"
-    />
+    /> -->
   </xacro:macro>
 </robot>
